Commit message: 0121添加了dual_ur5e的环境，能够在新的环境下邀操

File: assets/universal_robots_ur5e/dual_ur5e.urdf (robot description, URDF)
Before this commit: robot dual_ur5e_robot, 23 links, 22 joints
Links:
- added link base_link_robot, mass 400.99; collision mesh filename=file:///home/zz/mujoco_RL_file/robosuite/pico_vr/XRoboToolk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; visual mesh filename=file:///home/zz/mujoco_RL_file/robosuite/pico_vr/XRoboToolk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
- added link body_base_link, mass 5.3997; collision mesh filename=file:///home/zz/mujoco_RL_file/robosuite/pico_vr/XRoboToolk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; visual mesh filename=file:///home/zz/mujoco_RL_file/robosuite/pico_vr/XRoboToolk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
- added link body_left_base_link, mass 0.65565
- added link body_right_base_link, mass 0.65565
- added link bozi_link, mass 0.5717; collision mesh filename=file:///home/zz/mujoco_RL_file/robosuite/pico_vr/XRoboToolk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; visual mesh filename=file:///home/zz/mujoco_RL_file/robosuite/pico_vr/XRoboToolk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
- added link camera_fixed_link, mass 0.057939; collision mesh filename=file:///home/zz/mujoco_RL_file/robosuite/pico_vr/XRoboToolk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; visual mesh filename=file:///home/zz/mujoco_RL_file/robosuite/pico_vr/XRoboToolk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
- added link head_link, mass 2.8418; collision mesh filename=file:///home/zz/mujoco_RL_file/robosuite/pico_vr/XRoboToolk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; visual mesh filename=file:///home/zz/mujoco_RL_file/robosuite/pico_vr/XRoboToolk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
- added link left_correct_link
- added link left_dh_base_link, mass 0.407689241604604; collision mesh filename=file:///home/zz/mujoco_RL_file/robosuite/pico_vr/XRoboToolk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; visual mesh filename=file:///home/zz/mujoco_RL_file/robosuite/pico_vr/XRoboToolk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
- added link left_dh_center_link
- added link left_dh_finger1_link, mass 0.0589543896992846; collision mesh filename=file:///home/zz/mujoco_RL_file/robosuite/pico_vr/XRoboToolk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; visual mesh filename=file:///home/zz/mujoco_RL_file/robosuite/pico_vr/XRoboToolk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
- added link left_dh_finger2_link, mass 0.0589543896992846; collision mesh filename=file:///home/zz/mujoco_RL_file/robosuite/pico_vr/XRoboToolk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; visual mesh filename=file:///home/zz/mujoco_RL_file/robosuite/pico_vr/XRoboToolk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
- added link right_correct_link
- added link right_dh_base_link, mass 0.407689241604604; collision mesh filename=file:///home/zz/mujoco_RL_file/robosuite/pico_vr/XRoboToolk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; visual mesh filename=file:///home/zz/mujoco_RL_file/robosuite/pico_vr/XRoboToolk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
- added link right_dh_center_link
- added link right_dh_finger1_link, mass 0.0589543896992846; collision mesh filename=file:///home/zz/mujoco_RL_file/robosuite/pico_vr/XRoboToolk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; visual mesh filename=file:///home/zz/mujoco_RL_file/robosuite/pico_vr/XRoboToolk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
- added link right_dh_finger2_link, mass 0.0589543896992846; collision mesh filename=file:///home/zz/mujoco_RL_file/robosuite/pico_vr/XRoboToolk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; visual mesh filename=file:///home/zz/mujoco_RL_file/robosuite/pico_vr/XRoboToolk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
- added link world
Joints:
- added joint base_joint: type fixed, parent base_link, child base_link_robot, origin xyz=0.36 0 0 rpy=0.0 0.0 -1.5707963267948966
- added joint body_base_joint: type fixed, parent base_link, child body_base_link, origin xyz=0 0 0.78 rpy=0 0 1.5707963267948966
- added joint bozi_joint: type fixed, parent body_base_link, child bozi_link, origin xyz=-0.0468 -0.045 0.91925 rpy=1.5708 0 -1.5708
- added joint camera_fixed_joint: type fixed, parent head_link, child camera_fixed_link, origin xyz=0.10034 0.16948 -0.0168 rpy=-1.5708 0 -2.0943951
- added joint head_body_joint: type fixed, parent bozi_link, child head_link, origin xyz=0 0 0 rpy=0 0 -0.1
- added joint left_arm_fixed_joint: type fixed, parent body_base_link, child body_left_base_link, origin xyz=0.18182 0 0.63404 rpy=-0.95532 0.5236 -2.1863
- added joint left_correct_joint: type fixed, parent body_left_base_link, child left_correct_link, origin xyz=0 0 0 rpy=-1.5707963 -2.35619448975 0.0
- added joint left_dh_base_center_joint: type fixed, parent left_dh_base_link, child left_dh_center_link, origin xyz=0 0 0.14124 rpy=3.1416 -1.5708 0
- added joint left_dh_base_finger1_joint: type prismatic, parent left_dh_base_link, child left_dh_finger1_link, origin xyz=-0.0184 0.0 0.09325 rpy=0 0 -1.5708, axis -1 0 0, limit lower=0 upper=0.04 effort=30 velocity=0.5
- added joint left_dh_base_finger2_joint: type prismatic, parent left_dh_base_link, child left_dh_finger2_link, origin xyz=0.0184 -0.0 0.09325 rpy=0 0 1.5708, axis -1 0 0, limit lower=0 upper=0.04 effort=20 velocity=0.5, mimic joint=left_dh_base_finger1_joint multiplier=1 offset=0
- added joint left_gripper_joint: type fixed, parent left_tool0, child left_dh_base_link, origin xyz=0 0 0 rpy=0 0 -1.5707963
- added joint right_arm_fixed_joint: type fixed, parent body_base_link, child body_right_base_link, origin xyz=-0.17475 0 0.64111 rpy=-0.95532 -0.5236 2.1863
- added joint right_correct_joint: type fixed, parent body_right_base_link, child right_correct_link, origin xyz=0 0 0 rpy=-1.5707963 2.35619448975 0.0
- added joint right_dh_base_center_joint: type fixed, parent right_dh_base_link, child right_dh_center_link, origin xyz=0 0 0.14124 rpy=3.1416 -1.5708 0
- added joint right_dh_base_finger1_joint: type prismatic, parent right_dh_base_link, child right_dh_finger1_link, origin xyz=-0.0184 0.0 0.09325 rpy=0 0 -1.5708, axis -1 0 0, limit lower=0 upper=0.04 effort=30 velocity=0.5
- added joint right_dh_base_finger2_joint: type prismatic, parent right_dh_base_link, child right_dh_finger2_link, origin xyz=0.0184 -0.0 0.09325 rpy=0 0 1.5708, axis -1 0 0, limit lower=0 upper=0.04 effort=20 velocity=0.5, mimic joint=right_dh_base_finger1_joint multiplier=1 offset=0
- added joint right_gripper_joint: type fixed, parent right_tool0, child right_dh_base_link, origin xyz=0 0 0.006 rpy=0 0 -1.5707963
- added joint world_to_base_link: type fixed, parent world, child base_link, origin xyz=0 0 0 rpy=0 0 0
- joint world_to_left_arm_base: origin xyz=0 0.275 0.3 rpy=0.7853981633974483 0 3.141592653589793 -> xyz=0 0 0 rpy=00 0 0 ; parent base_link -> left_correct_link
- joint world_to_right_arm_base: origin xyz=0 -0.275 0.3 rpy=0.7853981633974483 0 0 -> xyz=0 0 0 rpy= 0 0 0 ; parent base_link -> right_correct_link

Commit message: 丰富了dual_ur5e的环境配置0122

File: assets/universal_robots_ur5e/dual_ur5e.urdf (robot description, URDF)
Before this commit: robot dual_ur5e_robot, 41 links, 40 joints
Joints:
- joint body_base_joint: origin xyz=0 0 0.78 rpy=0 0 1.5707963267948966 -> xyz=0 0 0.78 rpy=0 0 -1.5707963267948966
